File: Final_Proyect.kicad_sch (KiCad schematic)
At the start: 33 parts, among them J1 Conn_01x10_Pin, J2 VCC GND TTP223, J3 OLLED I2C, J4 - +, J5 USB_C, U1 ESP32-S3-WROOM-1, U2 AMS1117-3.3

Commit message: Actualizacion diseño PCB
Parts:
- added M_A1, M_B1, M_C1, M_D1, M_D2: VCC GND TTP223, Connector_JST:JST_EH_B2B-EH-A_1x02_P2.50mm_Vertical, symbol Connector:Conn_01x02_Pin
Connections:
- new net M1: M_A1.2 (Pin_2)
- new net M10: M_D1.1 (Pin_1)
- new net M2: M_A1.1 (Pin_1)
- new net M3: M_B1.2 (Pin_2)
- new net M4: M_B1.1 (Pin_1)
- new net M5: M_C1.2 (Pin_2)
- new net M6: M_C1.1 (Pin_1)
- new net M7: M_D2.2 (Pin_2)
- new net M8: M_D2.1 (Pin_1)
- new net M9: M_D1.2 (Pin_2)
- no-connect marks 0 -> 12
