File: Final_Proyect.kicad_pcb (KiCad board)
At the start: 2 copper layers, 66 x 52.5 mm, 77 parts, among them J1 Conn_01x10_Pin, J2 VCC GND TTP223, J4 - +, J5 USB_C, U1 ESP32-S3-WROOM-1, U2 AMS1117-3.3, U3 DRV8870DDA, U4 DRV8870DDA, U5 DRV8870DDA, U6 DRV8870DDA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

Commit message: Actualizacion diseño PCB
Parts:
- added ?: , , F.Cu at (158.5, 51.5)
- added ?: , , F.Cu at (111.5, 84.0)
- added J3: OLLED I2C, Connector_JST:JST_EH_B4B-EH-A_1x04_P2.50mm_Vertical, F.Cu at (164.5, 51.5)
- added M_A1: VCC GND TTP223, Connector_JST:JST_EH_B2B-EH-A_1x02_P2.50mm_Vertical, F.Cu at (110.5, 89.5)
- added M_B1: VCC GND TTP223, Connector_JST:JST_EH_B2B-EH-A_1x02_P2.50mm_Vertical, F.Cu at (119.0, 89.5)
- added M_C1: VCC GND TTP223, Connector_JST:JST_EH_B2B-EH-A_1x02_P2.50mm_Vertical, F.Cu at (127.5, 89.5)
- added M_D1: VCC GND TTP223, Connector_JST:JST_EH_B2B-EH-A_1x02_P2.50mm_Vertical, F.Cu at (136.0, 89.5)
- added M_D2: VCC GND TTP223, Connector_JST:JST_EH_B2B-EH-A_1x02_P2.50mm_Vertical, F.Cu at (144.8, 89.5)
- added REF**: MountingHole_3.2mm_M3_DIN965_Pad, MountingHole:MountingHole_3.2mm_M3_DIN965_Pad, F.Cu at (111.5, 46.0)
- added REF**: MountingHole_3.2mm_M3_DIN965_Pad, MountingHole:MountingHole_3.2mm_M3_DIN965_Pad, F.Cu at (158.5, 51.5)
- added REF**: MountingHole_3.2mm_M3_DIN965_Pad, MountingHole:MountingHole_3.2mm_M3_DIN965_Pad, F.Cu at (111.5, 84.0)
- moved J2 64.9 mm to (162.0, 89.5), turned to 0 degrees
- moved D1 57.1 mm to (158.0, 85.5), turned to 180 degrees
- moved R11 54.6 mm to (160.0, 83.5), turned to 180 degrees
- moved J4 49.5 mm to (153.5, 89.5), turned to 0 degrees
- moved C18 40.5 mm to (114.0, 66.5), turned to -90 degrees
- moved R32 40.5 mm to (108.0, 75.3)
- moved R33 40.4 mm to (109.5, 67.9), turned to -90 degrees
- moved R19 38.1 mm to (156.0, 81.6), turned to 90 degrees
- moved R41 37.9 mm to (122.1, 75.0)
- moved R34 35.6 mm to (109.5, 64.4), turned to 90 degrees
- moved R18 35.5 mm to (156.0, 76.3), turned to -90 degrees
- moved R20 35.3 mm to (141.0, 74.7)
- moved R21 34.9 mm to (144.5, 74.7)
- moved C7 34.8 mm to (147.9, 75.6)
- moved U3 34.8 mm to (151.9, 78.8)
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Connections:
- U3 pad 6: /Motor Driver/M1 -> /M1
- U3 pad 8: /Motor Driver/M2 -> /M2
- U4 pad 6: /Motor Driver1/M1 -> /M3
- U4 pad 8: /Motor Driver1/M2 -> /M4
- U5 pad 6: /Motor Driver2/M1 -> /M5
- U5 pad 8: /Motor Driver2/M2 -> /M6
- U6 pad 6: /Motor Driver3/M1 -> /M7
- U6 pad 8: /Motor Driver3/M2 -> /M8
- U7 pad 6: /Motor Driver4/M1 -> /M9
- U7 pad 8: /Motor Driver4/M2 -> /M10
Routing:
- net +3V3: track 37.3 -> 0.00 mm
- net D+: track 36.3 -> 0.00 mm
- net D-: track 35.6 -> 0.00 mm
- net BOOT: track 26.8 -> 0.00 mm, vias 2 -> 0
- net /Motor Driver2/IN2: track 25.6 -> 0.00 mm, vias 2 -> 0
- net F+: track 24.9 -> 0.00 mm, vias 2 -> 0
- net F-: track 21.9 -> 0.00 mm, vias 2 -> 0
- net C-: track 21.6 -> 0.00 mm, vias 2 -> 0
- net C+: track 19.4 -> 0.00 mm, vias 2 -> 0
- net /Motor Driver2/IN1: track 18.9 -> 0.00 mm, vias 2 -> 0
- net SIG10: track 16.6 -> 0.00 mm, vias 2 -> 0
- net /Motor Driver/IN2: track 16.3 -> 0.00 mm, vias 2 -> 0
- net /Motor Driver/IN1: track 16.3 -> 0.00 mm, vias 2 -> 0
- net SIG5: track 16.1 -> 0.00 mm, vias 2 -> 0
- net /Motor Driver1/IN2: track 15.8 -> 0.00 mm, vias 2 -> 0
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Other:
- board size 66 x 52.5 mm -> 60.5 x 52 mm
- board text added: "Final Proyect"
- board text added: "HandExo"
- board text added: "Rehab"

Commit message: Actualizacion de Drivers
Parts:
- moved R19 45.0 mm to (111.1, 79.5), turned to 0 degrees
- moved R17 44.5 mm to (108.5, 75.5), turned to -90 degrees
- moved R18 39.8 mm to (116.4, 79.5), turned to 180 degrees
- moved C8 39.5 mm to (110.0, 71.4), turned to 0 degrees
- moved U3 37.9 mm to (114.1, 75.4), turned to 0 degrees
- moved R21 36.8 mm to (108.5, 67.5), turned to 90 degrees
- moved R20 34.3 mm to (108.5, 64.0), turned to -90 degrees
- moved C9 32.2 mm to (113.5, 66.5), turned to -90 degrees
- moved C7 31.1 mm to (117.1, 71.4), turned to 180 degrees
- moved R35 26.5 mm to (136.8, 82.6), turned to 90 degrees
- moved R32 26.2 mm to (132.3, 85.0), turned to 0 degrees
- moved R34 22.5 mm to (121.4, 83.5), turned to 180 degrees
- moved R33 21.9 mm to (124.9, 83.5), turned to 0 degrees
- moved C17 21.7 mm to (128.3, 83.0), turned to 90 degrees
- moved R36 20.6 mm to (136.8, 76.5), turned to -90 degrees
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