File: PCB/PCB del Proyecto Final/Final_Proyect/Final_Proyect/Final_Proyect.kicad_sch (KiCad schematic)
At the start: 38 parts, among them J1 Conn_01x10_Pin, J2 VCC GND TTP223, J3 OLLED I2C, J4 - +, J5 USB_C, U1 ESP32-S3-WROOM-1, U2 AMS1117-3.3

Commit message: Version enrutada
Parts:
- removed M_A1, M_B1, M_C1, M_D1, M_D2: VCC GND TTP223, Connector_JST:JST_EH_B2B-EH-A_1x02_P2.50mm_Vertical, symbol Connector:Conn_01x02_Pin
- added J10, J6, J7, J8, J9: ~, Connector_JST:JST_EH_B2B-EH-A_1x02_P2.50mm_Vertical, symbol Connector:Conn_01x02_Pin
Connections:
- net SIG1: now also U1.38 (IO2); no longer U1.39 (IO1)
- net SIG2: now also U1.39 (IO1); no longer U1.38 (IO2)
- new net Motor Driver/M1: J6.1 (Pin_1)
- new net Motor Driver/M2: J6.2 (Pin_2)
- new net Motor Driver1/M1: J7.1 (Pin_1)
- new net Motor Driver1/M2: J7.2 (Pin_2)
- new net Motor Driver2/M1: J8.1 (Pin_1)
- new net Motor Driver2/M2: J8.2 (Pin_2)
- new net Motor Driver3/M1: J9.1 (Pin_1)
- new net Motor Driver3/M2: J9.2 (Pin_2)
- new net Motor Driver4/M1: J10.1 (Pin_1)
- new net Motor Driver4/M2: J10.2 (Pin_2)
- no-connect marks 12 -> 9
