File: PCB/DRB8870.kicad_sch (KiCad schematic)
At the start: 9 parts, among them U3 DRV8870DDA

Commit message: Enrutamiento mejorado
Parts:
- C7, C8: value C -> 100nF; LCSC (none) -> C519981
- C9: value C_Polarized -> 47uF; footprint Capacitor_SMD:CP_Elec_6.3x5.4 -> Capacitor_SMD:CP_Elec_6.3x7.7; LCSC (none) -> C7469965
- R17: value R -> 0.2; LCSC (none) -> C44051
- R18, R19: value R -> 1k; LCSC (none) -> C2907232
- R20: value R -> 80k; LCSC (none) -> C2960781
- R21: value R -> 10k
- U3: LCSC (none) -> C86590
Other:
- moved on the sheet: R17, R18, R19
Changed lines of the file:
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@@
 	(wire
 		(pts
-			(xy 99.06 96.52) (xy 100.33 96.52)
+			(xy 99.06 97.79) (xy 100.33 97.79)
 		)
 		(stroke
@@
 	(wire
 		(pts
-			(xy 99.06 100.33) (xy 100.33 100.33)
+			(xy 99.06 101.6) (xy 100.33 101.6)
 		)
 		(stroke
@@
 	(wire
 		(pts
-			(xy 107.95 96.52) (xy 110.49 96.52)
+			(xy 107.95 97.79) (xy 110.49 97.79)
 		)
 		(stroke
@@
 	(wire
 		(pts
-			(xy 107.95 100.33) (xy 110.49 100.33)
+			(xy 107.95 101.6) (xy 110.49 101.6)
 		)
 		(stroke
@@
 	(wire
 		(pts
-			(xy 97.79 90.17) (xy 99.06 90.17)
+			(xy 97.79 91.44) (xy 99.06 91.44)
 		)
 		(stroke
@@
 	(wire
 		(pts
-			(xy 107.95 90.17) (xy 106.68 90.17)
+			(xy 107.95 91.44) (xy 106.68 91.44)
 		)
 		(stroke
@@
 	)
 	(label "IN2"
-		(at 110.49 96.52 0)
+		(at 110.49 97.79 0)
 		(effects
 			(font
@@
 	)
 	(label "IN1"
-		(at 110.49 100.33 0)
+		(at 110.49 101.6 0)
 		(effects
 			(font
@@
 	)
 	(label "ISEN"
-		(at 97.79 90.17 180)
+		(at 97.79 91.44 180)
 		(effects
 			(font
@@
 	(hierarchical_label "IN.1"
 		(shape input)
-		(at 99.06 96.52 180)
+		(at 99.06 97.79 180)
 		(effects
 			(font
@@
 	(hierarchical_label "IN.2"
 		(shape input)
-		(at 99.06 100.33 180)
+		(at 99.06 101.6 180)
 		(effects
 			(font
@@
 			)
 		)
+		(property "LCSC" "C86590"
+			(at 176.53 99.06 0)
+			(effects
+				(font
+					(size 1.27 1.27)
+				)
+				(hide yes)
+			)
+		)
 		(pin "6"
 		)
@@
 			)
 		)
-		(property "Value" "R"
+		(property "Value" "10k"
 			(at 120.65 113.0299 0)
 			(effects
@@
 		)
 		(property "Description" "Resistor"
+			(at 118.11 111.76 0)
+			(effects
+				(font
+					(size 1.27 1.27)
+				)
+				(hide yes)
+			)
+		)
+		(property "LCSC" ""
 			(at 118.11 111.76 0)
 			(effects
@@
 			)
 		)
-		(property "Value" "C_Polarized"
+		(property "Value" "47uF"
 			(at 148.844 109.982 90)
 			(effects
@@
 			)
 		)
-		(property "Footprint" "Capacitor_SMD:CP_Elec_6.3x5.4"
+		(property "Footprint" "Capacitor_SMD:CP_Elec_6.3x7.7"
 			(at 145.7452 107.95 0)
 			(effects
@@
 		(property "Description" "Polarized capacitor"
 			(at 144.78 104.14 0)
+			(effects
+				(font
+					(size 1.27 1.27)
+				)
+				(hide yes)
+			)
+		)
+		(property "LCSC" "C7469965"
+			(at 144.78 104.14 90)
 			(effects
 				(font
@@
 	(symbol
 		(lib_id "power:GND")
-		(at 107.95 90.17 90)
+		(at 107.95 91.44 90)
 		(unit 1)
 		(exclude_from_sim no)
@@
 		(fields_autoplaced yes)
 		(property "Reference" "#PWR029"
-			(at 114.3 90.17 0)
+			(at 114.3 91.44 0)
 			(effects
 				(font
@@
 		)
 		(property "Value" "GND"
-			(at 111.76 90.1699 90)
+			(at 111.76 91.4399 90)
 			(effects
 				(font
@@
 		)
 		(property "Footprint" ""
-			(at 107.95 90.17 0)
+			(at 107.95 91.44 0)
 			(effects
 				(font
@@
 		)
 		(property "Datasheet" ""
-			(at 107.95 90.17 0)
+			(at 107.95 91.44 0)
 			(effects
 				(font
@@
 		)
 		(property "Description" "Power symbol creates a global label with name \"GND\" , ground"
-			(at 107.95 90.17 0)
+			(at 107.95 91.44 0)
 			(effects
 				(font
@@
 	(symbol
 		(lib_id "Device:R")
-		(at 102.87 90.17 90)
+		(at 102.87 91.44 90)
 		(unit 1)
 		(exclude_from_sim no)
@@
 		(fields_autoplaced yes)
 		(property "Reference" "R17"
-			(at 102.87 83.82 90)
-			(effects
-				(font
-					(size 1.27 1.27)
-				)
-			)
-		)
-		(property "Value" "R"
-			(at 102.87 86.36 90)
+			(at 102.87 85.09 90)
+			(effects
+				(font
+					(size 1.27 1.27)
+				)
+			)
+		)
+		(property "Value" "0.2"
+			(at 102.87 87.63 90)
 			(effects
 				(font
@@
 		)
 		(property "Footprint" "Resistor_SMD:R_1206_3216Metric"
-			(at 102.87 91.948 90)
+			(at 102.87 93.218 90)
 			(effects
 				(font
@@
 		)
 		(property "Datasheet" "~"
-			(at 102.87 90.17 0)
+			(at 102.87 91.44 0)
 			(effects
 				(font
@@
 		)
 		(property "Description" "Resistor"
-			(at 102.87 90.17 0)
+			(at 102.87 91.44 0)
+			(effects
+				(font
+					(size 1.27 1.27)
+				)
+				(hide yes)
+			)
+		)
+		(property "LCSC" "C44051"
+			(at 102.87 91.44 90)
 			(effects
 				(font
@@
 	(symbol
 		(lib_id "Device:R")
-		(at 104.14 96.52 90)
+		(at 104.14 97.79 90)
 		(unit 1)
 		(exclude_from_sim no)
@@
 		(dnp no)
 		(property "Reference" "R18"
-			(at 104.14 94.488 90)
-			(effects
-				(font
-					(size 1.27 1.27)
-				)
-			)
-		)
-		(property "Value" "R"
-			(at 104.14 96.52 90)
+			(at 104.14 95.758 90)
+			(effects
+				(font
+					(size 1.27 1.27)
+				)
+			)
+		)
+		(property "Value" "1k"
+			(at 104.14 97.79 90)
 			(effects
 				(font
@@
 		)
 		(property "Footprint" "Resistor_SMD:R_0805_2012Metric"
-			(at 104.14 98.298 90)
+			(at 104.14 99.568 90)
 			(effects
 				(font
@@
 		)
 		(property "Datasheet" "~"
-			(at 104.14 96.52 0)
+			(at 104.14 97.79 0)
 			(effects
 				(font
@@
 		)
 		(property "Description" "Resistor"
-			(at 104.14 96.52 0)
+			(at 104.14 97.79 0)
+			(effects
+				(font
+					(size 1.27 1.27)
+				)
+				(hide yes)
+			)
+		)
+		(property "LCSC" "C2907232"
+			(at 104.14 97.79 90)
 			(effects
 				(font
@@
 			)
 		)
-		(property "Value" "R"
+		(property "Value" "80k"
 			(at 120.65 101.5999 0)
 			(effects
@@
 		)
 		(property "Description" "Resistor"
+			(at 118.11 100.33 0)
+			(effects
+				(font
+					(size 1.27 1.27)
+				)
+				(hide yes)
+			)
+		)
+		(property "LCSC" "C2960781"
 			(at 118.11 100.33 0)
 			(effects
@@
 			)
 		)
-		(property "Value" "C"
+		(property "Value" "100nF"
 			(at 137.16 105.4099 0)
 			(effects
@@
 		)
 		(property "Description" "Unpolarized capacitor"
+			(at 133.35 104.14 0)
+			(effects
+				(font
+					(size 1.27 1.27)
+				)
+				(hide yes)
+			)
+		)
+		(property "LCSC" "C519981"
 			(at 133.35 104.14 0)
 			(effects
@@
 	(symbol
 		(lib_id "Device:R")
-		(at 104.14 100.33 270)
+		(at 104.14 101.6 270)
 		(unit 1)
 		(exclude_from_sim no)
@@
 		(dnp no)
 		(property "Reference" "R19"
-			(at 104.14 102.616 90)
-			(effects
-				(font
-					(size 1.27 1.27)
-				)
-			)
-		)
-		(property "Value" "R"
-			(at 104.14 100.33 90)
+			(at 104.14 103.886 90)
+			(effects
+				(font
+					(size 1.27 1.27)
+				)
+			)
+		)
+		(property "Value" "1k"
+			(at 104.14 101.6 90)
 			(effects
 				(font
@@
 		)
 		(property "Footprint" "Resistor_SMD:R_0805_2012Metric"
-			(at 104.14 98.552 90)
+			(at 104.14 99.822 90)
 			(effects
 				(font
@@
 		)
 		(property "Datasheet" "~"
-			(at 104.14 100.33 0)
+			(at 104.14 101.6 0)
 			(effects
 				(font
@@
 		)
 		(property "Description" "Resistor"
-			(at 104.14 100.33 0)
+			(at 104.14 101.6 0)
+			(effects
+				(font
+					(size 1.27 1.27)
+				)
+				(hide yes)
+			)
+		)
+		(property "LCSC" "C2907232"
+			(at 104.14 101.6 90)
 			(effects
 				(font
@@
 			)
 		)
-		(property "Value" "C"
+		(property "Value" "100nF"
 			(at 111.76 113.0299 0)
 			(effects
@@
 			(at 107.95 111.76 0)
 			(effects
+				(font
+					(size 1.27 1.27)
+				)
+				(hide yes)
+			)
+		)
+		(property "LCSC" "C519981"
+			(at 107.95 111.76 0)
+			(effects

Commit message: Finalizado
Parts:
- C7, C8: value 100nF -> 100nf; LCSC C519981 -> C710980
- C9: value 47uF -> 47uf; LCSC C7469965 -> C249753
- R17: LCSC C44051 -> C5127778
- R18, R19: LCSC C2907232 -> C2907295
- R20: LCSC C2960781 -> C2988920
- R21: LCSC (none) -> C2930231
Changed lines of the file:
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@@
 			)
 		)
-		(property "LCSC" ""
+		(property "LCSC" "C2930231"
 			(at 118.11 111.76 0)
 			(effects
@@
 			)
 		)
-		(property "Value" "47uF"
+		(property "Value" "47uf"
 			(at 148.844 109.982 90)
 			(effects
@@
 			)
 		)
-		(property "LCSC" "C7469965"
+		(property "LCSC" "C249753"
 			(at 144.78 104.14 90)
 			(effects
@@
 			)
 		)
-		(property "LCSC" "C44051"
+		(property "LCSC" "C5127778"
 			(at 102.87 91.44 90)
 			(effects
@@
 			)
 		)
-		(property "LCSC" "C2907232"
+		(property "LCSC" "C2907295"
 			(at 104.14 97.79 90)
 			(effects
@@
 			)
 		)
-		(property "LCSC" "C2960781"
+		(property "LCSC" "C2988920"
 			(at 118.11 100.33 0)
 			(effects
@@
 			)
 		)
-		(property "Value" "100nF"
+		(property "Value" "100nf"
 			(at 137.16 105.4099 0)
 			(effects
@@
 			)
 		)
-		(property "LCSC" "C519981"
+		(property "LCSC" "C710980"
 			(at 133.35 104.14 0)
 			(effects
@@
 			)
 		)
-		(property "LCSC" "C2907232"
+		(property "LCSC" "C2907295"
 			(at 104.14 101.6 90)
 			(effects
@@
 			)
 		)
-		(property "Value" "100nF"
+		(property "Value" "100nf"
 			(at 111.76 113.0299 0)
 			(effects
@@
 			)
 		)
-		(property "LCSC" "C519981"
+		(property "LCSC" "C710980"
 			(at 107.95 111.76 0)
 			(effects
